Commit message: updating the common color file, and the denso_arm_gazeob file

File: denso_arm/model/common.urdf.xacro (robot description, xacro)
@@ -1,24 +1,20 @@
+<?xml version="1.0" ?>
 <robot include-once="true" xmlns:xacro="http://ros.org/wiki/xacro">
+  <!-- Mathematical Constants -->
   <xacro:property name="PI" value="3.1415926535897931" />
-  <material name="denso_white">
-    <color rgba="1.0 1.0 1.0 1"/>
-  </material>
-  <material name="denso_light_gray">
-    <color rgba="0.8 0.8 0.8 1"/>
-  </material>
-  <material name="denso_med_gray">
-    <color rgba="0.6 0.6 0.6 1"/>
-  </material>
-  <material name="denso_dark_gray">
-    <color rgba="0.4 0.4 0.4 1"/>
-  </material>
-  <material name="denso_red">
-    <color rgba="0.5 0.4 0.4 1"/>
-  </material>
-  <material name="denso_green">
-    <color rgba="0.4 0.5 0.4 1"/>
-  </material>
-  <material name="denso_blue">
-    <color rgba="0.4 0.4 0.5 1"/>
-  </material>
+  <!-- Colors -->
+  <xacro:property name="DensoWhite"     value="1.0 1.0 1.0 1"/>
+  <xacro:property name="DensoLightGray" value="0.8 0.8 0.8 1"/>
+  <xacro:property name="DensoMedGray"   value="0.6 0.6 0.6 1"/>
+  <xacro:property name="DensoDarkGray"  value="0.4 0.4 0.4 1"/>
+  <xacro:property name="DensoRed"       value="0.5 0.4 0.4 1"/>
+  <xacro:property name="DensoGreen"     value="0.4 0.5 0.4 1"/>
+  <xacro:property name="DensoBlue"      value="0.4 0.4 0.5 1"/>
+  <material name="DensoWhite">    <color rgba="${DensoWhite}"/></material>
+  <material name="DensoLightGray"><color rgba="${DensoLightGray}"/></material>
+  <material name="DensoMedGray">  <color rgba="${DensoMedGray}"/></material>
+  <material name="DensoDarkGray"> <color rgba="${DensoDarkGray}"/></material>
+  <material name="DensoRed">      <color rgba="${DensoRed}"/></material>
+  <material name="DensoGreen">    <color rgba="${DensoGreen}"/></material>
+  <material name="DensoBlue">     <color rgba="${DensoBlue}"/></material>
 </robot>

File: denso_arm/model/denso_arm.urdf.xacro (robot description, xacro)
@@ -1,6 +1,5 @@
 <?xml version="1.0" ?>
 <robot
-<xmlns:xacro="http://www.ros.org/wiki/xacro"
-       name="denso_arm">
+  xmlns:xacro="http://www.ros.org/wiki/xacro">
   <material name="Grey">
     <color rgba="0.2 0.2 0.2 1.0"/>
@@ -13,5 +12,5 @@
       <origin xyz="0 0 0.098" rpy="0 0 0" />
       <geometry name="base_visual">
-	<box size="0.195 0.195 0.195" />
+	<mesh filename="package://denso_arm/meshes/" />
       </geometry>
       <material name="Grey" />
@@ -22,5 +21,5 @@
       <origin xyz="0 0 0.06" rpy="0 0 0" />
       <geometry name="link_1_visual">
-	<box size="0.100 0.100 0.120" />
+	<mesh filename="package://denso_arm/meshes" />
       </geometry>
       <material name="Grey" />
@@ -39,5 +38,5 @@
       <origin xyz="0 0 0.225" rpy="0 0 0" />
       <geometry name="link_2_visual">
-	<box size="0.05 0.05 0.400" />
+	<mesh filename="package://denso_arm/meshes" />
       </geometry>
       <material name="Grey" />
@@ -56,5 +55,5 @@
       <origin xyz="0 0 0.1425" rpy="0 0 0" />
       <geometry name="link_3_visual">
-	<box size="0.05 0.05 0.20" />
+	<mesh filename="package://denso_arm/meshes" />
       </geometry>
       <material name="Grey" />
@@ -73,5 +72,5 @@
       <origin xyz="0 0 0.0675" rpy="0 0 0" />
       <geometry name="link_4_visual">
-	<box size="0.05 0.05 0.10" />
+	<mesh filename="package://denso_arm/meshes" />
       </geometry>
       <material name="Grey" />
@@ -90,5 +89,5 @@
       <origin xyz="0 0 0.045" rpy="0 0 0" />
       <geometry name="link_5_visual">
-	<box size="0.03 0.03 0.08" />
+	<mesh filename="package://denso_arm/meshes" />
       </geometry>
       <material name="Grey" />
@@ -107,5 +106,5 @@
       <origin xyz="0 0 0.0005" rpy="0 0 0" />
       <geometry name="link_6_visual">
-	<box size="0.04 0.04 0.001" />
+	<mesh filename="package://denso_arm/meshes" />
       </geometry>
       <material name="LightGrey" />

File: denso_arm/model/denso_arm_gazebo.urdf.xacro (robot description, xacro)
@@ -13,7 +13,7 @@
       <origin xyz="0 0 0.098" rpy="0 0 0" />
       <geometry >
-	<mesh filename="package://denso_arm/meshes/" />
+        <mesh filename="package://denso_arm/meshes/" />
       </geometry>
-      <material name="denso_light_gray" />
+      <material name="DensoLightGray" />
     </visual>
      <inertial>
@@ -26,7 +26,7 @@
       <origin xyz="0 0 0.06" rpy="0 0 0" />
       <geometry >
-	<mesh filename="package://denso_arm/meshes" />
+        <mesh filename="package://denso_arm/meshes" />
       </geometry>
-      <material name="denso_light_gray" />
+      <material name="DensoLightGray" />
      </visual>
      <inertial>
@@ -41,5 +41,5 @@
     <axis xyz="0 0 1" />
     <limit lower="-2.967" upper="2.967" effort="10"
-	   velocity="1.0" />
+           velocity="1.0" />
     <joint_properties damping="0.0" friction="0.0"/>
   </joint>
@@ -48,5 +48,5 @@
       <origin xyz="0 0 0.225" rpy="0 0 0" />
       <geometry >
-	<mesh filename="package://denso_arm/meshes" />
+        <mesh filename="package://denso_arm/meshes" />
       </geometry>
       <material name="denso_med_gray" />
@@ -63,5 +63,5 @@
     <axis xyz="1 0 0" />
     <limit lower="-1.745" upper="2.356" effort="10"
-	   velocity="1.0" />
+           velocity="1.0" />
     <joint_properties damping="0.0" friction="0.0"/>
   </joint>
@@ -70,5 +70,5 @@
       <origin xyz="0 0 0.1425" rpy="0 0 0" />
       <geometry >
-	<mesh filename="package://denso_arm/meshes" />
+        <mesh filename="package://denso_arm/meshes" />
       </geometry>
       <material name="denso_dark_gray" />
@@ -85,5 +85,5 @@
     <axis xyz="1 0 0" />
     <limit lower="-2.094" upper="2.670" effort="10"
-	   velocity="1.0" />
+           velocity="1.0" />
     <joint_properties damping="0.0" friction="0.0"/>
   </joint>
@@ -92,7 +92,7 @@
       <origin xyz="0 0 0.0675" rpy="0 0 0" />
       <geometry >
-	<mesh filename="package://denso_arm/meshes" />
+        <mesh filename="package://denso_arm/meshes" />
       </geometry>
-      <material name="denso_light_gray" />
+      <material name="DensoLightGray" />
     </visual>
        <inertial>
@@ -107,5 +107,5 @@
     <axis xyz="0 0 1" />
     <limit lower="-4.712" upper="4.712" effort="10"
-	   velocity="1.0" />
+           velocity="1.0" />
     <joint_properties damping="0.0" friction="0.0"/>
  </joint>
@@ -114,7 +114,7 @@
       <origin xyz="0 0 0.045" rpy="0 0 0" />
       <geometry >
-	<mesh filename="package://denso_arm/meshes" />
+        <mesh filename="package://denso_arm/meshes" />
       </geometry>
-      <material name="denso_light_gray" />
+      <material name="DensoLightGray" />
     </visual>
        <inertial>
@@ -129,5 +129,5 @@
     <axis xyz="1 0 0" />
     <limit lower="-2.094" upper="2.094" effort="10"
-	   velocity="1.0" />
+           velocity="1.0" />
     <joint_properties damping="0.0" friction="0.0"/>
   </joint>
@@ -136,7 +136,7 @@
       <origin xyz="0 0 0.0005" rpy="0 0 0" />
       <geometry >
-	<mesh filename="package://denso_arm/meshes" />
+        <mesh filename="package://denso_arm/meshes" />
       </geometry>
-      <material name="denso_light_gray" />
+      <material name="DensoLightGray" />
     </visual>
        <inertial>
@@ -151,5 +151,5 @@
     <axis xyz="0 0 1" />
     <limit lower="-6.283" upper="6.283" effort="10"
-	   velocity="1.0" />
+           velocity="1.0" />
     <joint_properties damping="0.0" friction="0.0"/>
   </joint>
