Commit message: revisions so that package can be used specifically with Ros Hydro and catkin

File: denso_arm/model/denso_arm_gazebo.urdf.xacro (robot description, xacro)
@@ -1,17 +1,18 @@
 <?xml version="1.0" ?>
-<robot
-  xmlns:xacro="http://www.ros.org/wiki/xacro">
+<!-- Denso 6DOF Manipulator-->
+<robot name="denso" xmlns:xacro="http://www.ros.org/wiki/xacro">
+  <!-- ros_control plugin-->
   <gazebo>
       <plugin name="ros_control" filename="libros_control_gazebo_plugin.so">
-        <ns>denso/ros_control</ns>
-        <robotSimType>ros_control_gazebo_tests/MTMSim</robotSimType>
-        <controlPeriod>0.001</controlPeriod>
+        <robotNamespace>/denso</robotNamespace>
       </plugin>
     </gazebo>
+    <!-- Import all Gazebo-customization elements, including Gazebo colors -->
+   <xacro:include filename="$(find denso_arm)/model/common.urdf.xacro" />
   <link name="base">
     <visual>
       <origin xyz="0 0 0.098" rpy="0 0 0" />
       <geometry >
-        <mesh filename="package://denso_arm/meshes/" />
+        <mesh filename="package://denso_arm/meshes/denso_1Link.stl" />
       </geometry>
       <material name="DensoLightGray" />
@@ -26,5 +27,5 @@
       <origin xyz="0 0 0.06" rpy="0 0 0" />
       <geometry >
-        <mesh filename="package://denso_arm/meshes" />
+        <mesh filename="package://denso_arm/meshes/denso_2Link.stl" />
       </geometry>
       <material name="DensoLightGray" />
@@ -48,5 +49,5 @@
       <origin xyz="0 0 0.225" rpy="0 0 0" />
       <geometry >
-        <mesh filename="package://denso_arm/meshes" />
+        <mesh filename="package://denso_arm/meshes/denso_3Link.stl" />
       </geometry>
       <material name="denso_med_gray" />
@@ -70,5 +71,5 @@
       <origin xyz="0 0 0.1425" rpy="0 0 0" />
       <geometry >
-        <mesh filename="package://denso_arm/meshes" />
+        <mesh filename="package://denso_arm/meshes/denso_4Link.stl" />
       </geometry>
       <material name="denso_dark_gray" />
@@ -92,5 +93,5 @@
       <origin xyz="0 0 0.0675" rpy="0 0 0" />
       <geometry >
-        <mesh filename="package://denso_arm/meshes" />
+        <mesh filename="package://denso_arm/meshes/denso_5Link.stl" />
       </geometry>
       <material name="DensoLightGray" />
@@ -114,5 +115,5 @@
       <origin xyz="0 0 0.045" rpy="0 0 0" />
       <geometry >
-        <mesh filename="package://denso_arm/meshes" />
+        <mesh filename="package://denso_arm/meshes/denso_6Link.stl" />
       </geometry>
       <material name="DensoLightGray" />
@@ -132,25 +133,3 @@
     <joint_properties damping="0.0" friction="0.0"/>
   </joint>
-  <link name="link_6">
-    <visual>
-      <origin xyz="0 0 0.0005" rpy="0 0 0" />
-      <geometry >
-        <mesh filename="package://denso_arm/meshes" />
-      </geometry>
-      <material name="DensoLightGray" />
-    </visual>
-       <inertial>
-        <mass value="2"/>
-        <inertia ixx="2.0" ixy="0.0" ixz="0.0" iyy="2.0" iyz="0.0" izz="2.0"/>
-      </inertial>
-  </link>
-  <joint name="denso_J5" type="revolute">
-    <parent link="link_5"/>
-    <child link="link_6"/>
-    <origin xyz="0 0 0.090" rpy="0 0 0" />
-    <axis xyz="0 0 1" />
-    <limit lower="-6.283" upper="6.283" effort="10"
-           velocity="1.0" />
-    <joint_properties damping="0.0" friction="0.0"/>
-  </joint>
 </robot>
