Commit message: working package just need to modify the linkagesand implement the stl files

File: denso_arm/model/denso_box.urdf.xacro (robot description, xacro)
@@ -2,13 +2,14 @@
 <!-- Denso 6DOF Manipulator-->
 <robot name="denso" xmlns:xacro="http://www.ros.org/wiki/xacro">
-  <!-- ros_control plugin-->
-  <gazebo>
-      <plugin name="gazebo_ros_control" filename="libros_control_gazebo_plugin.so">
-        <robotNamespace>/denso</robotNamespace>
-      </plugin>
-    </gazebo>
-    <!-- Import all Gazebo-customization elements, including Gazebo colors -->
-   <xacro:include filename="$(find denso_arm)/model/common.urdf.xacro" />
-  <link name="base">
+     <!-- Import all Gazebo-customization elements, including Gazebo colors -->
+ <xacro:include filename="$(find denso_arm)/model/denso.gazebo" />
+         <!-- Import Rviz colors -->
+ <xacro:include filename="$(find denso_arm)/model/materials.xacro" />
+<link name = "world"/>
+<joint name="fixed" type="fixed">
+    <parent link="world"/>
+    <child link="link1"/>
+</joint>
+<link name="link1">
     <visual>
       <origin xyz="0 0 0.098" rpy="0 0 0" />
@@ -16,12 +17,14 @@
        <box size="0.195 0.195 0.195" />
       </geometry>
-      <material name="DensoLightGray" />
+      <material name="orange" />
     </visual>
      <inertial>
         <mass value="9"/>
-        <inertia ixx="9.0" ixy="0.0" ixz="0.0" iyy="9.0" iyz="0.0" izz="9.0"/>
+        <inertia ixx="9.0" ixy="0.0" ixz="0.0"
+                 iyy="9.0" iyz="0.0"
+                 izz="9.0"/>
       </inertial>
   </link>
-  <link name="link_1">
+  <link name="link2">
     <visual>
       <origin xyz="0 0 0.06" rpy="0 0 0" />
@@ -29,5 +32,5 @@
      <box size="0.100 0.100 0.120" />
       </geometry>
-      <material name="DensoLightGray" />
+      <material name="black" />
      </visual>
      <inertial>
@@ -37,6 +40,6 @@
   </link>
   <joint name="denso_J0" type="revolute">
-    <parent link="base"/>
-    <child link="link_1"/>
+    <parent link="link1"/>
+    <child link="link2"/>
     <origin xyz="0 0 0.198" rpy="0 0 1.57" />
     <axis xyz="0 0 1" />
@@ -45,5 +48,5 @@
     <joint_properties damping="0.0" friction="0.0"/>
   </joint>
-  <link name="link_2">
+  <link name="link3">
     <visual>
       <origin xyz="0 0 0.225" rpy="0 0 0" />
@@ -51,5 +54,5 @@
         <box size="0.05 0.05 0.400" />
       </geometry>
-      <material name="denso_med_gray" />
+      <material name="orange" />
     </visual>
         <inertial>
@@ -59,6 +62,6 @@
   </link>
   <joint name="denso_J1" type="revolute">
-    <parent link="link_1"/>
-    <child link="link_2"/>
+    <parent link="link2"/>
+    <child link="link3"/>
     <origin xyz="0 0 0.190" rpy="0 0 0" />
     <axis xyz="1 0 0" />
@@ -67,86 +70,19 @@
     <joint_properties damping="0.0" friction="0.0"/>
   </joint>
-  <link name="link_3">
-    <visual>
-      <origin xyz="0 0 0.1425" rpy="0 0 0" />
-      <geometry >
-        <box size="0.05 0.05 0.20" />
-      </geometry>
-      <material name="denso_dark_gray" />
-    </visual>
-    <inertial>
-        <mass value="6"/>
-        <inertia ixx="6.0" ixy="0.0" ixz="0.0" iyy="6.0" iyz="0.0" izz="6.0"/>
-      </inertial>
-  </link>
-  <joint name="denso_J2" type="revolute">
-    <parent link="link_2"/>
-    <child link="link_3"/>
-    <origin xyz="0 0 0.450" rpy="0 0 0" />
-    <axis xyz="1 0 0" />
-    <limit lower="-2.094" upper="2.670" effort="10"
-           velocity="1.0" />
-    <joint_properties damping="0.0" friction="0.0"/>
-  </joint>
-  <link name="link_4">
-    <visual>
-      <origin xyz="0 0 0.0675" rpy="0 0 0" />
-      <geometry >
-       <box size="0.05 0.05 0.10" />
-      </geometry>
-      <material name="DensoLightGray" />
-    </visual>
-       <inertial>
-        <mass value="5"/>
-        <inertia ixx="5.0" ixy="0.0" ixz="0.0" iyy="5.0" iyz="0.0" izz="5.0"/>
-      </inertial>
-  </link>
-  <joint name="denso_J3" type="revolute">
-    <parent link="link_3"/>
-    <child link="link_4"/>
-    <origin xyz="0 0 0.285" rpy="0 0 0" />
-    <axis xyz="0 0 1" />
-    <limit lower="-4.712" upper="4.712" effort="10"
-           velocity="1.0" />
-    <joint_properties damping="0.0" friction="0.0"/>
- </joint>
-  <link name="link_5">
-    <visual>
-      <origin xyz="0 0 0.045" rpy="0 0 0" />
-      <geometry >
-        <box size="0.03 0.03 0.08" />
-      </geometry>
-      <material name="DensoLightGray" />
-    </visual>
-       <inertial>
-        <mass value="4"/>
-        <inertia ixx="4.0" ixy="0.0" ixz="0.0" iyy="4.0" iyz="0.0" izz="4.0"/>
-      </inertial>
-  </link>
-  <joint name="denso_J4" type="revolute">
-    <parent link="link_4"/>
-    <child link="link_5"/>
-    <origin xyz="0 0 0.135" rpy="0 0 0" />
-    <axis xyz="1 0 0" />
-    <limit lower="-2.094" upper="2.094" effort="10"
-           velocity="1.0" />
-    <joint_properties damping="0.0" friction="0.0"/>
-  </joint>
- <link name="link_6">
-     <visual>
-    <origin xyz="0 0 0.0005" rpy="0 0 0" />
-       <geometry >
-     <box size="0.04 0.04 0.001" />
-       </geometry>
-        <material name="DensoLightGrey" />
-       </visual>
-   </link>
-     <joint name="denso_J5" type="revolute">
-         <parent link="link_5"/>
-         <child link="link_6"/>
-         <origin xyz="0 0 0.090" rpy="0 0 0" />
-          <axis xyz="0 0 1" />
-        <limit lower="-6.283" upper="6.283" effort="10"
-                         velocity="1.0" />
-    </joint>
+<transmission name="tran1">
+    <type>transmission_interface/SimpleTransmission</type>
+    <joint name="joint1"/>
+    <actuator name="motor1">
+       <hardwareInterface>EffortJointInterface</hardwareInterface>
+       <mechanicalReduction>1</mechanicalReduction>
+     </actuator>
+ </transmission>
+   <transmission name="tran2">
+       <type>transmission_interface/SimpleTransmission</type>
+       <joint name="joint2"/>
+       <actuator name="motor2">
+         <hardwareInterface>EffortJointInterface</hardwareInterface>
+         <mechanicalReduction>1</mechanicalReduction>
+      </actuator>
+   </transmission>
 </robot>

Commit message: current working denso simulation, where each link is represented by a rectangular box

File: denso_arm/model/denso_box.urdf.xacro (robot description, xacro)
@@ -15,5 +15,5 @@
       <origin xyz="0 0 0.098" rpy="0 0 0" />
       <geometry >
-       <box size="0.195 0.195 0.195" />
+      <box size="0.195 0.195 0.195" />
       </geometry>
       <material name="orange" />
@@ -28,7 +28,7 @@
   <link name="link2">
     <visual>
-      <origin xyz="0 0 0.06" rpy="0 0 0" />
+            <origin xyz="0 0 0.06" rpy="0 0 0" />
       <geometry >
-     <box size="0.100 0.100 0.120" />
+       <box size="0.100 0.100 0.120" />
       </geometry>
       <material name="black" />
@@ -39,8 +39,8 @@
       </inertial>
   </link>
-  <joint name="denso_J0" type="revolute">
+  <joint name="joint1" type="revolute">
     <parent link="link1"/>
     <child link="link2"/>
-    <origin xyz="0 0 0.198" rpy="0 0 1.57" />
+       <origin xyz="0 0 0.198" rpy="0 0 1.57" />
     <axis xyz="0 0 1" />
     <limit lower="-2.967" upper="2.967" effort="10"
@@ -50,7 +50,7 @@
   <link name="link3">
     <visual>
-      <origin xyz="0 0 0.225" rpy="0 0 0" />
+       <origin xyz="0 0 0.225" rpy="0 0 0" />
       <geometry >
-        <box size="0.05 0.05 0.400" />
+      <box size="0.05 0.05 0.400" />
       </geometry>
       <material name="orange" />
@@ -61,11 +61,99 @@
       </inertial>
   </link>
-  <joint name="denso_J1" type="revolute">
+  <joint name="joint2" type="revolute">
     <parent link="link2"/>
     <child link="link3"/>
-    <origin xyz="0 0 0.190" rpy="0 0 0" />
+      <origin xyz="0 0 0.190" rpy="0 0 0" />
     <axis xyz="1 0 0" />
     <limit lower="-1.745" upper="2.356" effort="10"
            velocity="1.0" />
+    <joint_properties damping="0.0" friction="0.0"/>
+  </joint>
+  <link name="link4">
+    <visual>
+            <origin xyz="0 0 0.1425" rpy="0 0 0" />
+      <geometry >
+      <box size="0.05 0.05 0.20" />
+      </geometry>
+      <material name="orange" />
+    </visual>
+        <inertial>
+        <mass value="7"/>
+        <inertia ixx="7.0" ixy="0.0" ixz="0.0" iyy="7.0" iyz="0.0" izz="7.0"/>
+      </inertial>
+  </link>
+  <joint name="joint3" type="revolute">
+    <parent link="link3"/>
+    <child link="link4"/>
+     <origin xyz="0 0 0.450" rpy="0 0 0" />
+    <axis xyz="1 0 0" />
+     <limit lower="-2.094" upper="2.670" effort="10"
+                velocity="1.0" />
+    <joint_properties damping="0.0" friction="0.0"/>
+  </joint>
+  <link name="link5">
+    <visual>
+      <origin xyz="0 0 0.0675" rpy="0 0 0" />
+      <geometry >
+       <box size="0.05 0.05 0.10" />
+      </geometry>
+      <material name="orange" />
+    </visual>
+        <inertial>
+        <mass value="7"/>
+        <inertia ixx="7.0" ixy="0.0" ixz="0.0" iyy="7.0" iyz="0.0" izz="7.0"/>
+      </inertial>
+  </link>
+  <joint name="joint4" type="revolute">
+    <parent link="link4"/>
+    <child link="link5"/>
+    <origin xyz="0 0 0.285" rpy="0 0 0" />
+    <axis xyz="1 0 0" />
+    <limit lower="-4.712" upper="4.712" effort="10"
+               velocity="1.0" />
+    <joint_properties damping="0.0" friction="0.0"/>
+  </joint>
+  <link name="link6">
+    <visual>
+       <origin xyz="0 0 0.045" rpy="0 0 0" />
+      <geometry >
+      <box size="0.03 0.03 0.08" />
+      </geometry>
+      <material name="orange" />
+    </visual>
+        <inertial>
+        <mass value="7"/>
+        <inertia ixx="7.0" ixy="0.0" ixz="0.0" iyy="7.0" iyz="0.0" izz="7.0"/>
+      </inertial>
+  </link>
+  <joint name="joint5" type="revolute">
+    <parent link="link5"/>
+    <child link="link6"/>
+    <origin xyz="0 0 0.135" rpy="0 0 0" />
+        <axis xyz="1 0 0" />
+    <limit lower="-2.094" upper="2.094" effort="10"
+               velocity="1.0" />
+    <joint_properties damping="0.0" friction="0.0"/>
+  </joint>
+  <link name="link7">
+    <visual>
+      <origin xyz="0 0 0.0005" rpy="0 0 0" />
+      <geometry >
+        <box size="0.04 0.04 0.001" />
+      </geometry>
+      <material name="orange" />
+    </visual>
+        <inertial>
+        <mass value="7"/>
+        <inertia ixx="7.0" ixy="0.0" ixz="0.0" iyy="7.0" iyz="0.0" izz="7.0"/>
+      </inertial>
+  </link>
+  <joint name="joint6" type="revolute">
+    <parent link="link6"/>
+    <child link="link7"/>
+     <origin xyz="0 0 0.090" rpy="0 0 0" />
+         <axis xyz="0 0 1" />
+             <limit lower="-6.283" upper="6.283" effort="10"
+                        velocity="1.0" />
     <joint_properties damping="0.0" friction="0.0"/>
   </joint>
